File: CabHat_relay.kicad_pcb (KiCad board)
At the start: 2 copper layers, 100 x 70 mm, 4 parts

Commit message: v1.00
Parts:
- added C1: 100n, Library:C_0603_1608Metric, F.Cu at (148.0, 90.1)
- added D1: D, Library:D_SOD-123, F.Cu at (144.7, 103.5)
- added D2: D, Library:D_SOD-123, F.Cu at (162.4, 103.5)
- added D3: D, Library:D_SOD-123, F.Cu at (180.2, 103.5)
- added D4: D, Library:D_SOD-123, F.Cu at (190.9, 65.2)
- added D5: D, Library:D_SOD-123, F.Cu at (173.1, 65.2)
- added D6: D, Library:D_SOD-123, F.Cu at (155.3, 65.2)
- added D7: D, Library:D_SOD-123, F.Cu at (137.6, 65.2)
- added D8: D, Library:D_SOD-123, F.Cu at (119.8, 65.2)
- added J1: Barrel_Jack_Switch, Library:BarrelJack_GCT_DCJ200-10-A_Horizontal, F.Cu at (114.4, 85.0)
- added J10: Screw_Terminal_01x03, Library:TerminalBlock_akizuki_TB111_P5.08mm, F.Cu at (132.2, 54.5)
- added J11: Screw_Terminal_01x03, Library:TerminalBlock_akizuki_TB111_P5.08mm, F.Cu at (114.4, 54.5)
- added J2: Conn_01x08, Library:PinSocket_1x08_P2.54mm_Vertical, F.Cu at (110.0, 110.0)
- added J3: Conn_01x04, Library:Grove_1x04_P2mm_Horizontal_silk_inside, F.Cu at (108.0, 100.2)
- added J4: Screw_Terminal_01x03, Library:TerminalBlock_akizuki_TB111_P5.08mm, F.Cu at (150.0, 115.5)
- added J5: Screw_Terminal_01x03, Library:TerminalBlock_akizuki_TB111_P5.08mm, F.Cu at (167.8, 115.5)
- added J6: Screw_Terminal_01x03, Library:TerminalBlock_akizuki_TB111_P5.08mm, F.Cu at (185.6, 115.5)
- added J7: Screw_Terminal_01x03, Library:TerminalBlock_akizuki_TB111_P5.08mm, F.Cu at (185.6, 54.5)
- added J8: Screw_Terminal_01x03, Library:TerminalBlock_akizuki_TB111_P5.08mm, F.Cu at (167.8, 54.5)
- added J9: Screw_Terminal_01x03, Library:TerminalBlock_akizuki_TB111_P5.08mm, F.Cu at (150.0, 54.5)
- added JP1: SolderJumper_2_Open, Library:SolderJumper-2_P1.3mm_Open_RoundedPad1.0x1.5mm, F.Cu at (114.4, 93.9)
- added JP2: SolderJumper_2_Open, Library:SolderJumper-2_P1.3mm_Open_RoundedPad1.0x1.5mm, B.Cu at (147.2, 91.9)
- added JP3: SolderJumper_2_Open, Library:SolderJumper-2_P1.3mm_Open_RoundedPad1.0x1.5mm, B.Cu at (150.0, 91.9)
- added JP4: SolderJumper_2_Open, Library:SolderJumper-2_P1.3mm_Open_RoundedPad1.0x1.5mm, B.Cu at (152.8, 91.9)
- added K1: Y14x-1C-xxDS, Library:Relay_SPDT_HsinDa_Y14, F.Cu at (147.5, 107.8)
- added K2: Y14x-1C-xxDS, Library:Relay_SPDT_HsinDa_Y14, F.Cu at (165.3, 107.8)
- added K3: Y14x-1C-xxDS, Library:Relay_SPDT_HsinDa_Y14, F.Cu at (183.1, 107.8)
- added K4: Y14x-1C-xxDS, Library:Relay_SPDT_HsinDa_Y14, F.Cu at (188.0, 61.0)
- added K5: Y14x-1C-xxDS, Library:Relay_SPDT_HsinDa_Y14, F.Cu at (170.2, 61.0)
- added K6: Y14x-1C-xxDS, Library:Relay_SPDT_HsinDa_Y14, F.Cu at (152.5, 61.0)
- added K7: Y14x-1C-xxDS, Library:Relay_SPDT_HsinDa_Y14, F.Cu at (134.7, 61.0)
- added K8: Y14x-1C-xxDS, Library:Relay_SPDT_HsinDa_Y14, F.Cu at (116.9, 61.0)
- added LED1: LED, Library:LED_0603_1608Metric, F.Cu at (140.6, 99.5)
- added LED2: LED, Library:LED_0603_1608Metric, F.Cu at (158.4, 99.5)
- added LED3: LED, Library:LED_0603_1608Metric, F.Cu at (176.2, 99.5)
- added LED4: LED, Library:LED_0603_1608Metric, F.Cu at (195.0, 69.3)
- added LED5: LED, Library:LED_0603_1608Metric, F.Cu at (177.2, 69.3)
- added LED6: LED, Library:LED_0603_1608Metric, F.Cu at (159.4, 69.3)
- added LED7: LED, Library:LED_0603_1608Metric, F.Cu at (141.6, 69.3)
- added LED8: LED, Library:LED_0603_1608Metric, F.Cu at (123.8, 69.3)
- added Q1: Q_NMOS_GSD, Library:SOT-23, F.Cu at (141.6, 103.0)
- added Q2: Q_NMOS_GSD, Library:SOT-23, F.Cu at (159.4, 103.0)
- added Q3: Q_NMOS_GSD, Library:SOT-23, F.Cu at (177.2, 103.0)
- added Q4: Q_NMOS_GSD, Library:SOT-23, F.Cu at (193.9, 65.7)
- added Q5: Q_NMOS_GSD, Library:SOT-23, F.Cu at (176.2, 65.7)
- added Q6: Q_NMOS_GSD, Library:SOT-23, F.Cu at (158.4, 65.7)
- added Q7: Q_NMOS_GSD, Library:SOT-23, F.Cu at (140.6, 65.7)
- added Q8: Q_NMOS_GSD, Library:SOT-23, F.Cu at (122.8, 65.7)
- added R1: 10k, Library:R_0603_1608Metric, F.Cu at (147.2, 93.1)
- added R10: 10k, Library:R_0603_1608Metric, F.Cu at (139.6, 69.3)
- added R11: 10k, Library:R_0603_1608Metric, F.Cu at (121.8, 69.3)
- added R2: 10k, Library:R_0603_1608Metric, F.Cu at (150.0, 93.1)
- added R3: 10k, Library:R_0603_1608Metric, F.Cu at (152.8, 93.1)
- added R4: 10k, Library:R_0603_1608Metric, F.Cu at (142.6, 99.5)
- added R5: 10k, Library:R_0603_1608Metric, F.Cu at (160.4, 99.5)
- added R6: 10k, Library:R_0603_1608Metric, F.Cu at (178.2, 99.5)
- added R7: 10k, Library:R_0603_1608Metric, F.Cu at (192.9, 69.3)
- added R8: 10k, Library:R_0603_1608Metric, F.Cu at (175.1, 69.3)
- added R9: 10k, Library:R_0603_1608Metric, F.Cu at (157.4, 69.3)
- added U1: PCA9555PW, Library:TSSOP-24_4.4x7.8mm_P0.65mm, F.Cu at (150.0, 85.0)
Routing:
- net GND: track 0.00 -> 307.2 mm, vias 0 -> 8
- net +VSW: track 0.00 -> 229.1 mm, vias 0 -> 7
- net +3V3: track 0.00 -> 66.1 mm, vias 0 -> 1
- net /SDA: track 0.00 -> 57.7 mm, vias 0 -> 1
- net ex.IO0_3: track 0.00 -> 56.4 mm
- net /SCL: track 0.00 -> 55.3 mm, vias 0 -> 1
- net ex.IO0_7: track 0.00 -> 52.0 mm
- net ex.IO0_2: track 0.00 -> 43.7 mm
- net ex.IO0_4: track 0.00 -> 37.0 mm
- net ex.IO0_6: track 0.00 -> 36.3 mm
- net +5V: track 0.00 -> 34.3 mm
- net ex.IO0_0: track 0.00 -> 30.0 mm
- net ex.IO0_1: track 0.00 -> 26.4 mm
- net /relay02/COM: track 0.00 -> 22.6 mm
- net /relay01/COM: track 0.00 -> 22.6 mm
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- added copper zone on B.Cu, net GND
- added copper zone on F.Cu, net GND
- removed copper zone on B.Cu, net (none)
- removed copper zone on F.Cu, net (none)
Other:
- board text added: "${TITLE} Rev. ${REVISION} ${ISSUE_DATE} Designed by ${COMPANY} Lot: JLCJLCJLCJLC"
- board text added: "A0"
- board text added: "A1"
- board text added: "A2"
- board text added: "address:0b0100"
- board text added: "short:1 open:0"
