File: CabHat_relay.kicad_sch (KiCad schematic)
At the start: 10 parts, among them J1 Conn_01x04, J19 Barrel_Jack_Switch, J2 Conn_01x08, U1 PCA9555PW

Commit message: v1.00
Parts:
- removed J19: Barrel_Jack_Switch, Connector_BarrelJack:BarrelJack_GCT_DCJ200-10-A_Horizontal, symbol Library:Barrel_Jack_Switch
- added C1: 100n, Library:C_0603_1608Metric, symbol Library:C
- added J1: Barrel_Jack_Switch, Library:BarrelJack_GCT_DCJ200-10-A_Horizontal, symbol Connector:Barrel_Jack_Switch
- added JP1: SolderJumper_2_Open, Library:SolderJumper-2_P1.3mm_Open_RoundedPad1.0x1.5mm, symbol Library:SolderJumper_2_Open
- J2: footprint Connector_PinSocket_2.54mm:PinSocket_1x05_P2.54mm_Vertical -> Library:PinSocket_1x08_P2.54mm_Vertical
- J3: renamed from J1; footprint 0-myLibrary:Grove_1x04_P2mm_Horizontal_silk_inside -> Library:Grove_1x04_P2mm_Horizontal_silk_inside
- JP2: renamed from JP1; footprint Jumper:SolderJumper-2_P1.3mm_Bridged_RoundedPad1.0x1.5mm -> Library:SolderJumper-2_P1.3mm_Open_RoundedPad1.0x1.5mm
- JP3: renamed from JP2; footprint Jumper:SolderJumper-2_P1.3mm_Bridged_RoundedPad1.0x1.5mm -> Library:SolderJumper-2_P1.3mm_Open_RoundedPad1.0x1.5mm
- JP4: renamed from JP3; footprint Jumper:SolderJumper-2_P1.3mm_Bridged_RoundedPad1.0x1.5mm -> Library:SolderJumper-2_P1.3mm_Open_RoundedPad1.0x1.5mm
- R1, R2, R3: footprint Resistor_SMD:R_0603_1608Metric -> Library:R_0603_1608Metric
- U1: footprint Package_SO:TSSOP-24_4.4x7.8mm_P0.65mm -> Library:TSSOP-24_4.4x7.8mm_P0.65mm
Connections:
- net +3V3: now also C1.1
- net +5V: now also JP1.1 (A)
- net +VSW: now also J1.1, JP1.2 (B)
- net GND: now also C1.2, J1.2, J1.3
- no-connect marks 4 -> 12
Other:
- removed sheet relay10
- removed sheet relay11
- removed sheet relay12
- removed sheet relay13
- removed sheet relay14
- removed sheet relay15
- removed sheet relay16
- removed sheet relay17
- moved on the sheet: J3
