File: relay.kicad_sch (KiCad schematic)
At the start: 6 parts, among them J4 Screw_Terminal_01x03, K1 Y14x-1C-xxDS, Q1 Q_NMOS_GSD

Commit message: v1.00
Parts:
- D1: footprint (none) -> Library:D_SOD-123; lcsc C2128 -> C81598
- J4: footprint TerminalBlock:TerminalBlock_bornier-3_P5.08mm -> Library:TerminalBlock_akizuki_TB111_P5.08mm; lcsc (none) -> x
- K1: footprint Relay_THT:Relay_SPDT_HsinDa_Y14 -> Library:Relay_SPDT_HsinDa_Y14
- LED1: footprint LED_SMD:LED_0603_1608Metric -> Library:LED_0603_1608Metric
- Q1: footprint Package_TO_SOT_SMD:SOT-23 -> Library:SOT-23
- R4: footprint Resistor_SMD:R_0603_1608Metric -> Library:R_0603_1608Metric; lcsc C23162 -> C25804
Connections:
- net N.C.: now also J4.3 (Pin_3); no longer J4.1 (Pin_1)
- net N.O.: now also J4.1 (Pin_1); no longer J4.3 (Pin_3)
Other:
- company: (none) -> @stop_pattern
- title: (none) -> CabHat_relay
Changed lines of the file:
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@@
 (kicad_sch (version 20211123) (generator eeschema)
   (paper "A4")
+  (title_block
+    (title "CabHat_relay")
+    (rev "1.00")
+    (company "@stop_pattern")
+  )
   (junction (at 139.7 63.5) (diameter 0) (color 0 0 0 0)
   )
@@
     (stroke (width 0) (type default) (color 0 0 0 0))
   )
-  (label "N.C." (at 190.5 73.66 0)
+  (label "N.C." (at 190.5 78.74 0)
     (effects (font (size 1.27 1.27)) (justify left bottom))
   )
@@
     (effects (font (size 1.27 1.27)) (justify left bottom))
   )
-  (label "N.O." (at 190.5 78.74 0)
+  (label "N.O." (at 190.5 73.66 0)
     (effects (font (size 1.27 1.27)) (justify left bottom))
   )
@@
       (effects (font (size 1.27 1.27)) (justify right))
     )
-    (property "Footprint" "LED_SMD:LED_0603_1608Metric" (id 2) (at 127 127 0)
+    (property "Footprint" "Library:LED_0603_1608Metric" (id 2) (at 127 127 0)
       (effects (font (size 1.27 1.27)) hide)
     )
@@
       (effects (font (size 1.27 1.27)) (justify left))
     )
-    (property "Footprint" "Resistor_SMD:R_0603_1608Metric" (id 2) (at 125.222 114.3 90)
+    (property "Footprint" "Library:R_0603_1608Metric" (id 2) (at 125.222 114.3 90)
       (effects (font (size 1.27 1.27)) hide)
     )
@@
       (effects (font (size 1.27 1.27)) hide)
     )
-    (property "lcsc" "C23162" (id 4) (at 127 114.3 0)
+    (property "lcsc" "C25804" (id 4) (at 127 114.3 0)
       (effects (font (size 1.27 1.27)) hide)
     )
@@
   (symbol (lib_id "power:+VSW") (at 139.7 57.15 0) (unit 1)
     (in_bom yes) (on_board yes) (fields_autoplaced)
-    (property "Reference" "#PWR021" (id 0) (at 139.7 60.96 0)
+    (property "Reference" "#PWR024" (id 0) (at 139.7 60.96 0)
       (effects (font (size 1.27 1.27)) hide)
     )
@@
       (effects (font (size 1.27 1.27)) (justify left))
     )
-    (property "Footprint" "" (id 2) (at 133.35 76.2 0)
+    (property "Footprint" "Library:D_SOD-123" (id 2) (at 133.35 76.2 0)
       (effects (font (size 1.27 1.27)) hide)
     )
@@
       (effects (font (size 1.27 1.27)) hide)
     )
-    (property "lcsc" "C2128" (id 4) (at 133.35 76.2 0)
+    (property "lcsc" "C81598" (id 4) (at 133.35 76.2 0)
       (effects (font (size 1.27 1.27)) hide)
     )
@@
   (symbol (lib_id "power:GND") (at 139.7 133.35 0) (unit 1)
     (in_bom yes) (on_board yes) (fields_autoplaced)
-    (property "Reference" "#PWR022" (id 0) (at 139.7 139.7 0)
+    (property "Reference" "#PWR025" (id 0) (at 139.7 139.7 0)
       (effects (font (size 1.27 1.27)) hide)
     )
@@
       (effects (font (size 1.27 1.27)) (justify left))
     )
-    (property "Footprint" "Package_TO_SOT_SMD:SOT-23" (id 2) (at 142.24 99.06 0)
+    (property "Footprint" "Library:SOT-23" (id 2) (at 142.24 99.06 0)
       (effects (font (size 1.27 1.27)) hide)
     )
@@
       (effects (font (size 1.27 1.27)) (justify left))
     )
-    (property "Footprint" "TerminalBlock:TerminalBlock_bornier-3_P5.08mm" (id 2) (at 203.2 76.2 0)
+    (property "Footprint" "Library:TerminalBlock_akizuki_TB111_P5.08mm" (id 2) (at 203.2 76.2 0)
       (effects (font (size 1.27 1.27)) hide)
     )
@@
       (effects (font (size 1.27 1.27)) hide)
     )
+    (property "lcsc" "x" (id 4) (at 203.2 76.2 0)
+      (effects (font (size 1.27 1.27)) hide)
+    )
     (pin "1")
     (pin "2")
@@
   (symbol (lib_id "power:GND") (at 127 133.35 0) (unit 1)
     (in_bom yes) (on_board yes) (fields_autoplaced)
-    (property "Reference" "#PWR020" (id 0) (at 127 139.7 0)
+    (property "Reference" "#PWR023" (id 0) (at 127 139.7 0)
       (effects (font (size 1.27 1.27)) hide)
     )
@@
       (effects (font (size 1.27 1.27)) (justify left))
     )
-    (property "Footprint" "Relay_THT:Relay_SPDT_HsinDa_Y14" (id 2) (at 163.83 77.47 0)
+    (property "Footprint" "Library:Relay_SPDT_HsinDa_Y14" (id 2) (at 163.83 77.47 0)
       (effects (font (size 1.27 1.27)) (justify left) hide)
     )
